File: _autosave-1Cell_LiPO_BOOST_converter.kicad_pcb (KiCad board)
At the start: 2 copper layers, 40 x 40 mm, 39 parts, among them J1 microUSB, J4 USB_A, Q1 BC847, Q2 BC847, SW1 ON/OFF, U1 MCP73831, U2 MCP1661

Commit message: Added Rev B
Parts:
- removed REF**: KiCad-Logo2_6mm_SilkScreen, Symbol:KiCad-Logo2_6mm_SilkScreen
- removed REF**: OSHW-Symbol_6.7x6mm_SilkScreen, Symbol:OSHW-Symbol_6.7x6mm_SilkScreen
- moved D1 8.26 mm to (142.2, 116.8)
- moved R3 1.42 mm to (146.1, 118.1)
Connections:
- D1 pad 1: GND -> Net-(D1-Pad1)
- R3 pad 1: Net-(R3-Pad1) -> Net-(BATT1-Pad1)
- U1 pad 1: Net-(R3-Pad1) -> Net-(D1-Pad1)
Routing:
- net Net-(BATT1-Pad1): track 43.5 -> 51.3 mm, vias 1 -> 3
- net Net-(R3-Pad1): track 7.25 -> 0.00 mm, vias 2 -> 0
- net Net-(D1-Pad2): track 9.55 -> 3.79 mm
- net Net-(D1-Pad1): track 0.00 -> 1.91 mm
- net Net-(R12-Pad2): track 28.9 -> 30.5 mm
- net GND: vias 8 -> 7
Other:
- board text added: "1 cell LiPO BOOST converter By Martynas J. 19-03-03 Rev B"
- board text removed: "1 cell LiPO BOOST converter By Martynas J. 19-02-01 Rev A"
